File: handheld1_motion4sim_FO41AFC70E184.kicad_sch (KiCad schematic)
At the start: 16 parts, among them J1 RJ45, J2 Conn_01x03, J3 Conn_01x06, Q1 AO3400A, Q2 AO3400A, Q3 AO3400A

Commit message: shoaib
Parts:
- removed D1, D2: ESD9B3.3ST5G, Diode_SMD:D_SOD-923, symbol Diode:ESD9B3.3ST5G
- added JP1: Jumper_2_Open, Jumper:SolderJumper-2_P1.3mm_Open_Pad1.0x1.5mm, symbol Jumper:Jumper_2_Open
- J1: footprint Connector_RJ:RJ45_OST_PJ012-8P8CX_Vertical -> Connector_RJ:RJ45_Molex_0855135013_Vertical; LCSC (none) -> C708653
- J2: LCSC (none) -> C161870
- J3: LCSC (none) -> C161873
- Q1, Q2, Q3: LCSC (none) -> C20917
- R1, R2, R3: footprint (none) -> Resistor_SMD:R_0402_1005Metric; LCSC (none) -> C25076
- R4, R5, R6: footprint (none) -> Resistor_SMD:R_0402_1005Metric; LCSC (none) -> C25530
Connections:
- net LED_GREEN: now also R1.1; no longer R2.1
- net LED_YELLOW: now also R2.1; no longer R1.1
- net Y_cathode: now also JP1.2 (B); no longer Q3.3 (D)
- net at Q2.1 (G), R5.2: now also R1.2; no longer R2.2
- net at Q3.1 (G), R4.2: now also R2.2; no longer R1.2
- new net: JP1.1 (A), Q3.3 (D)
Other:
- note added: "-Active LOW -5V -No current Limiting necessary -Have connection but not using yellow - The LEDS have builtin resistors"
- note removed: "-Active LOW -5V -No current Limiting necessary -Have connection but not using yellow"
